File: ChuaCircuits.kicad_sch (KiCad schematic)
At the start: 23 parts, among them J1 BanaJack 9V, J2 BanaJack GND, J3 BanaJack -9V, U1 TL082, U2 TL082

Commit message: first connection tests
Parts:
- C1, C2, C3: footprint (none) -> Capacitor_THT:C_Disc_D7.5mm_W5.0mm_P7.50mm
- C4, C5, C6, C7: footprint (none) -> Capacitor_THT:C_Disc_D3.8mm_W2.6mm_P2.50mm
- R1, R2, R3, R4, R5, R6, R7, R8, R9: footprint (none) -> PCM_Resistor_THT_AKL:R_Axial_DIN0207_L6.3mm_D2.5mm_P10.16mm_Horizontal
- U1, U2: footprint (none) -> Package_DIP:DIP-8_W7.62mm

Commit message: finished board v1
Parts:
- removed J1: BanaJack 9V, Connector:Banana_Jack_1Pin, symbol Connector:Conn_01x01_Pin
- removed J2: BanaJack GND, Connector:Banana_Jack_1Pin, symbol Connector:Conn_01x01_Pin
- removed J3: BanaJack -9V, Connector:Banana_Jack_1Pin, symbol Connector:Conn_01x01_Pin
- added H1, H2, H3, H4: MountingHole_Pad, MountingHole:MountingHole_2.7mm_M2.5_DIN965_Pad, symbol Mechanical:MountingHole_Pad
- added J1: PWR_Input, addons:1985205, symbol Connector:Conn_01x03_Socket
- added J2, J3: Output_1, addons:1985205, symbol Connector:Conn_01x03_Socket
Connections:
- net +9V: now also J1.3 (Pin_3)
- net -9V: now also J1.1 (Pin_1)
- net GND: now also H1.1, H2.1, H3.1, H4.1, J1.2 (Pin_2), J2.3 (Pin_3), J3.2 (Pin_2), J3.3 (Pin_3)
- net X-Value: now reaches C1.1, R1.2, R4.1, RV1.1, U2.3 (+), U2.5 (+)
- net X-Value: now also J2.1 (Pin_1)
- net at R8.2, R9.1, U1.2 (-): now also U1.6 (-); no longer U1.5 (+)
- net Y-Value: now reaches C2.1, R7.1, RV1.2, U1.3 (+)
- net Y-Value: now also J2.2 (Pin_2)
- net at C3.2, RV2.1: now also U1.5 (+); no longer U1.6 (-)
- net Z-Value: now reaches R7.2, R8.1, U1.7
- net Z-Value: now also J3.1 (Pin_1)
